File: TM-001-60-2.kicad_pcb (KiCad board)
At the start: 2 copper layers, 24 parts, among them SW1 SW_Push, U1 ATmega32U4-AU, Y1 16MHz

Commit message: Routing donezo
whether it's any good or not i'm yet to see
Parts:
- moved C7 6.40 mm to (57.1, 66.7), turned to 270 degrees
- moved C1 3.97 mm to (71.9, 44.9)
- moved C2 3.97 mm to (61.8, 44.9)
- moved Y1 3.97 mm to (66.8, 44.9)
- moved R1 1.12 mm to (56.2, 52.9), turned to 270 degrees
- moved C4 1.12 mm to (59.4, 52.9)
- moved D3 0.79 mm to (98.4, 67.5), turned to 90 degrees
- moved D4 0.79 mm to (117.5, 67.5), turned to 90 degrees
- moved D1 0.79 mm to (98.4, 48.4), turned to 90 degrees
- moved D2 0.79 mm to (117.5, 48.4), turned to 90 degrees
- turned F1 to 90 degrees
Connections:
- U1 pad 27: Net-(U1-Pad27) -> ROW0
- U1 pad 28: Net-(U1-Pad28) -> COL1
- U1 pad 29: Net-(U1-Pad29) -> COL0
- U1 pad 30: Net-(U1-Pad30) -> ROW1
Routing:
- net GND: track 0.00 -> 154.7 mm
- net +5V: track 0.00 -> 110.8 mm, vias 0 -> 5
- net ROW1: track 0.00 -> 54.4 mm
- net COL1: track 0.00 -> 54.0 mm
- net ROW0: track 0.00 -> 51.7 mm
- net COL0: track 0.00 -> 34.6 mm
- net Net-(R1-Pad2): track 0.00 -> 30.0 mm, vias 0 -> 2
- net Net-(R3-Pad1): track 0.00 -> 27.6 mm
- net Net-(R2-Pad1): track 0.00 -> 26.5 mm
- net Net-(C2-Pad1): track 0.00 -> 17.9 mm
- net Net-(C1-Pad1): track 0.00 -> 14.6 mm
- net VCC: track 0.00 -> 9.84 mm
- net Net-(D2-Pad2): track 0.00 -> 6.72 mm
- net Net-(D1-Pad2): track 0.00 -> 6.72 mm
- net Net-(D4-Pad2): track 0.00 -> 6.72 mm
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Other:
- net class Default: trace_width 0.25 -> 0.254
- net class Power added: clearance 0.2, trace_width 0.381, via_dia 0.8, via_drill 0.4

Commit message: nearly finished pcb
just need to get all the errors to stop coming up and i'll be well away
Parts:
- moved C5 1.46 mm to (74.6, 57.1)
- moved C6 1.27 mm to (72.1, 69.8)
- moved C1 1.27 mm to (70.6, 44.9)
- moved C2 0.95 mm to (62.7, 44.9)
Routing:
- net GND: track 154.7 -> 146.4 mm
- net +5V: track 110.8 -> 106.2 mm
- net Net-(C1-Pad1): track 14.6 -> 13.3 mm
- net Net-(C2-Pad1): track 17.9 -> 16.9 mm
- added copper zone on B.Cu, net GND
Other:
- board outline added: 79.4 x 38.1 mm
- board text added: ":nice:"
